File: circuits/projects/Power_board/power_board.sch (EAGLE design)
At the start: 5 parts

Commit message: circuit board work
Parts:
- removed BATTERY-1, BATTERY-2: (no value), iStivi - Header-Connector:M02-1.5MM
- removed E-STOP, ON-OFF: 2-PIN-SWITCH2X1.5MM_HOLES, iStivi - Button-Switch:2-PIN-SWITCH2X1.5MM_HOLES
- added BATTERY1, BATTERY2: 12V, parts:BATTERY-ST
- added C1: 10uF, parts:CAPACITOR
- added C2: 2.2uF, parts:CAPACITOR
- added DIODE30A: NTST30100SG-H, parts:NTST30100SG-H
- added M1-FUSE, M2-FUSE: 20A, parts:FUSE
- added MOBO+12V: 2-HOLESSC3.81MM, parts:2-HOLESSC3.81MM
- added MOTOR-1, MOTOR-2: 2-HOLESSC5MM, parts:2-HOLESSC5MM
- added RELAY-1, RELAY-2: 5V, parts:RT424A05
- added VR-1: LT323A, parts:LT323AT-V
- CHARGER: value (none) -> 2-HOLESSC5MM; device iStivi - Header-Connector:M02-1.5MM -> parts:2-HOLESSC5MM
Connections:
- removed net VCC: BATTERY-1.1, ON-OFF.2
- new net N$1: BATTERY1.+, C2.1, RELAY-12.P, RELAY-13.P, VR-1.IN
- new net N$10: M2-FUSE.1, MOTOR-2.2
- new net N$4: CHARGER.2, DIODE30A.A, RELAY-11.1, RELAY-13.S, RELAY-21.1
- new net N$5: BATTERY2.+, RELAY-23.P
- new net N$6: RELAY-12.O
- new net N$7: DIODE30A.C, RELAY-23.S
- new net N$8: C1.1, MOBO+12V.2, VR-1.OUT
- new net N$9: M1-FUSE.1, MOTOR-1.2
- net GND: now also BATTERY1.-, C1.2, C2.2, CHARGER.1, MOBO+12V.1, MOTOR-1.1, MOTOR-2.1, RELAY-11.2, RELAY-21.2, RELAY-22.S, VR-1.GND; no longer BATTERY-2.2, CHARGER.2
- net N$2: now also BATTERY2.-, RELAY-13.O, RELAY-22.P; no longer E-STOP.2, ON-OFF.1
- net N$3: now also M1-FUSE.2, M2-FUSE.2, RELAY-23.O; no longer BATTERY-1.2, BATTERY-2.1
Other:
- note added: "+12V"
- note added: "+24V"
- note added: "0V"
- note added: "Battery Charger Relay switches"
- note added: "Drive motors"
- note added: "Motherboard Always powered"
- moved on the sheet: CHARGER

Commit message: board work
Parts:
- removed DIODE30A: NTST30100SG-H, parts:NTST30100SG-H
- removed RELAY-1, RELAY-2: 5V, parts:RT424A05
- removed VR-1: LT323A, parts:LT323AT-V
- added 12V_REG1, 12V_REG2, 5V_1, 5V_2, 5V_3, 5V_4: 2-HOLESSC3.81MM, parts:2-HOLESSC3.81MM
- added BATT1_V, BATT2_V: 1-HOLE, parts:1-HOLE
- added C10, C13, C14, C7, C8, C9: 0.1uF, parts:CAPACITOR_POL
- added C11, C12, C3, C4, C5: 0.33uF, parts:CAPACITOR_POL
- added C6: (no value), parts:CAPACITOR_POL
- added D1-12V, D2-12V, D3-24V: 30A, parts:NTST30100SG-H
- added IC1, IC2: (no value), parts:L7812CD2T-TRTO-263
- added RELAY: 5V, parts:RT424A05
- added RELAY_ON: 1-HOLE", parts:1-HOLE"
- added VR1: LT323A, parts:LT323AT-V
- added VR2, VR3, VR4, VR5: L7805, parts:L7805ACD2T-TR
- CHARGER: value 2-HOLESSC5MM -> 24V
Connections:
- new net N$11: RELAY1.1, RELAY_ON.1
- new net N$12: C2.1, D2-12V.C, VR1.IN
- new net N$13: 5V_2.2, VR3.OUT
- new net N$14: 5V_3.2, VR4.OUT
- new net N$15: 5V_4.2, VR5.OUT
- new net N$16: C3.+, C4.+, C5.+, D1-12V.C, VR2.IN, VR3.IN, VR4.IN, VR5.IN
- new net N$17: 12V_REG1.1, IC1.OUT
- new net N$18: 12V_REG2.1, C14.+, IC2.OUT
- net GND: now also 12V_REG1.2, 12V_REG2.2, 5V_1.1, 5V_2.1, 5V_3.1, 5V_4.1, C10.-, C11.-, C12.-, C13.-, C14.-, C3.-, C4.-, C5.-, C7.-, C8.-, C9.-, IC1.GND, IC2.GND, RELAY1.2, VR1.GND, VR2.GND, VR3.GND, VR4.GND, VR5.GND; no longer RELAY-11.2, RELAY-21.2, RELAY-22.S, VR-1.GND
- net N$1: now also BATT1_V.1, BATTERY2.-, D2-12V.A, RELAY2.P; no longer C2.1, RELAY-12.P, RELAY-13.P, VR-1.IN
- net N$2: now also CHARGER.2, RELAY3.S; no longer BATTERY2.-, RELAY-13.O, RELAY-22.P
- net N$3: now also C12.+, D3-24V.C, IC1.IN, IC2.IN; no longer RELAY-23.O
- net N$4: now also D3-24V.A, RELAY3.O; no longer CHARGER.2, DIODE30A.A, RELAY-11.1, RELAY-13.S, RELAY-21.1
- net N$5: now also BATT2_V.1, RELAY3.P; no longer RELAY-23.P
- net N$6: now also D1-12V.A, RELAY2.O; no longer RELAY-12.O
- net N$7: now also 5V_1.2, VR2.OUT; no longer DIODE30A.C, RELAY-23.S
- net N$8: now also VR1.OUT; no longer VR-1.OUT
Other:
- note added: "Regulated 12V 1.5A"
- note added: "Regulated 5V 1A"
- moved on the sheet: C1, C2, MOBO+12V

Commit message: circuits and charger plans
Parts:
- removed 12V_REG1, 12V_REG2: 2-HOLESSC3.81MM, parts:2-HOLESSC3.81MM
- removed IC1, IC2: (no value), parts:L7812CD2T-TRTO-263
- removed VR1: LT323A, parts:LT323AT-V
- removed VR2, VR3, VR4, VR5: L7805, parts:L7805ACD2T-TR
- added 12V-1, 12V-2, 12V-3, 12V_AM1, 12V_AM2, 12V_REG-1, 12V_REG-2, 12V_SERVO1, 12V_SERVO2, 12V_SERVO3, 12V_SERVO4, 12V_SERVO5, 12V_SERVO6: 2-HOLESSC3.81MM, parts:2-HOLESSC3.81MM
- added C15, C17, C19, C21, C23, C25, C28, C30: 0.1uF, parts:CAPACITOR_POL
- added C16, C18, C20, C22, C24, C26, C27, C29: 0.33uF, parts:CAPACITOR_POL
- added R10, R12, R14, R16, R6, R8: 1K, parts:RESISTOR0207/2V
- added R11, R13, R15, R5, R7, R9: 270R, parts:RESISTOR0207/2V
- added U$7, U$8: FUSEBLADE, parts:FUSEBLADE
- added VR-12-1: l7812, parts:L7812CD2T-TRTO-263
- added VR-12-2: L7812, parts:L7812CD2T-TRTO-263
- added VR-5-1, VR-5-2, VR-5-3, VR-5-4: L7805, parts:L7805ACD2T-TR
- added VR-A-1, VR-A-2: LM1085-12V, parts:LM1085IT-V
- added VR-MB: LT323A, parts:LT323AT-V
- added VR-S1, VR-S2, VR-S3, VR-S4, VR-S5, VR-S6: LM338T-V, parts:LM338T-V
- C6: value (none) -> 0.33uF
Connections:
- removed net N$16: C3.+, C4.+, C5.+, D1-12V.C, VR2.IN, VR3.IN, VR4.IN, VR5.IN
- new net N$19: R5.2, R6.1, VR-S1.ADJ
- new net N$20: RELAY3.P, U$7.2
- new net N$21: 12V_REG-2.2, C30.+, VR-12-1.OUT
- new net N$22: C12.+, C16.+, C26.+, D3-24V.C, M1-FUSE.2, M2-FUSE.2, VR-A-1.IN, VR-A-2.IN, VR-S1.IN, VR-S6.IN
- new net N$23: 12V_SERVO1.2, C15.+, R5.1, VR-S1.OUT
- new net N$24: C18.+, VR-S2.IN
- new net N$25: 12V_SERVO2.2, C17.+, R7.1, VR-S2.OUT
- new net N$26: R7.2, R8.1, VR-S2.ADJ
- new net N$27: C20.+, VR-S3.IN
- new net N$28: 12V_SERVO3.2, C19.+, R9.1, VR-S3.OUT
- new net N$29: R10.1, R9.2, VR-S3.ADJ
- new net N$30: C22.+, VR-S4.IN
- new net N$31: 12V_SERVO4.2, C21.+, R11.1, VR-S4.OUT
- new net N$32: R11.2, R12.1, VR-S4.ADJ
- new net N$33: C24.+, VR-S5.IN
- new net N$34: 12V_SERVO5.2, C23.+, R13.1, VR-S5.OUT
- new net N$35: R13.2, R14.1, VR-S5.ADJ
- new net N$36: 12V-1.2, 12V-2.2, 12V-3.2, C3.+, C4.+, C5.+, C6.+, D1-12V.C, VR-5-1.IN, VR-5-2.IN, VR-5-3.IN, VR-5-4.IN
- new net N$37: 12V_SERVO6.2, C25.+, R15.1, VR-S6.OUT
- new net N$38: R15.2, R16.1, VR-S6.ADJ
- new net N$39: RELAY2.P, U$8.1
- new net N$40: 12V_SERVO2.1, C17.-, C18.-, R8.2
- new net N$44: 12V_SERVO6.1, C25.-, C26.-, R16.2
- net GND: now also 12V-1.1, 12V-2.1, 12V-3.1, 12V_AM1.1, 12V_AM2.1, 12V_REG-1.1, 12V_REG-2.1, 12V_SERVO1.1, 12V_SERVO3.1, 12V_SERVO4.1, 12V_SERVO5.1, C15.-, C16.-, C19.-, C20.-, C21.-, C22.-, C23.-, C24.-, C27.+, C27.-, C29.+, C29.-, C30.-, C6.-, R10.2, R12.2, R14.2, R6.2, VR-12-1.GND, VR-12-1.IN, VR-12-2.GND, VR-12-2.IN, VR-5-1.GND, VR-5-2.GND, VR-5-3.GND, VR-5-4.GND, VR-A-1.GND, VR-A-2.GND, VR-MB.GND; no longer 12V_REG1.2, 12V_REG2.2, IC1.GND, IC2.GND, VR1.GND, VR2.GND, VR3.GND, VR4.GND, VR5.GND
- net N$1: now also U$8.2; no longer RELAY2.P
- net N$12: now also VR-MB.IN; no longer VR1.IN
- net N$13: now also VR-5-2.OUT; no longer VR3.OUT
- net N$14: now also VR-5-3.OUT; no longer VR4.OUT
- net N$15: now also C10.+, VR-5-4.OUT; no longer VR5.OUT
- net N$17: now also 12V_AM1.2, VR-A-1.OUT; no longer 12V_REG1.1, IC1.OUT
- net N$18: now also 12V_AM2.2, VR-A-2.OUT; no longer 12V_REG2.1, IC2.OUT
- net N$3: now also 12V_REG-1.2, C28.+, VR-12-2.OUT; no longer C12.+, D3-24V.C, IC1.IN, IC2.IN, M1-FUSE.2, M2-FUSE.2
- net N$5: now also U$7.1; no longer RELAY3.P
- net N$7: now also VR-5-1.OUT; no longer VR2.OUT
- net N$8: now also VR-MB.OUT; no longer VR1.OUT
Other:
- note added: "12V 3A Servo Motor Power"
- note added: "12V Unregulated"
- note added: "Regulated 12V 3A Actuator Motors"
- moved on the sheet: 5V_1, 5V_2, 5V_3, 5V_4, BATT1_V, BATT2_V, BATTERY1, BATTERY2, C1, C10, C11, C12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
