File: circuits/projects/Power_board/distribution_board.sch (EAGLE design)
At the start: 73 parts

Commit message: new board and some ignores
Parts:
- removed C11, C12, C16, C18, C20, C22, C24, C26, C27, C29, C3, C4, C5, C6: 0.33uF, parts:CAPACITOR_POL
- added C_12V, C_5V, C_ACT, C_SERVO1, C_SERVO2: 0.33uF, parts:CAPACITOR_POL
- INPUT, OUTPUT: value 3-HOLES -> (none)
- VR-A-1, VR-A-2: device parts:LM1085IT-V -> parts:LM1085IT-SINK
- VR-S1, VR-S2, VR-S3, VR-S4, VR-S5, VR-S6: value LM338T-V -> LM338T-SINK; device parts:LM338T-V -> parts:LM338T-SINK
Connections:
- net 12V: now also C_5V.+; no longer C3.+, C4.+, C5.+, C6.+
- net 24V: now also C_12V.+, C_ACT.+, C_SERVO1.+, C_SERVO2.+; no longer C12.+, C16.+, C18.+, C20.+, C22.+, C24.+, C26.+, C27.+, C29.+
- net GND: now also C28.-, C_12V.-, C_5V.-, C_ACT.-, C_SERVO1.-, C_SERVO2.-; no longer C11.-, C12.-, C16.-, C18.-, C20.-, C22.-, C24.-, C26.-, C27.-, C29.-, C3.-, C4.-, C5.-, C6.-
- net N$13: now also C8.+
- net N$14: now also C9.+
- net N$17: now also C13.+
- net N$7: now also C7.+

Commit message: gittin the night away
Parts:
- 12V-1, 12V-2, 12V-3, 12V_AM1, 12V_AM2, 12V_REG-1, 12V_REG-2, 12V_SERVO1, 12V_SERVO2, 12V_SERVO3, 12V_SERVO4, 12V_SERVO5, 12V_SERVO6, 5V_1, 5V_2, 5V_3, 5V_4: value 2-HOLESSC3.81MM -> SC3.81MM
- INPUT, OUTPUT: value (none) -> SC3.8MM
- VR-12-1: value l7812 -> L7812
Changed lines of the file:
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@@
 <setting verticaltext="up"/>
 </settings>
-<grid distance="0.05" unitdist="inch" unit="inch" style="lines" multiple="1" display="no" altdistance="0.025" altunitdist="inch" altunit="inch"/>
+<grid distance="0.1" unitdist="inch" unit="inch" style="lines" multiple="1" display="no" altdistance="0.01" altunitdist="inch" altunit="inch"/>
 <layers>
 <layer number="1" name="Top" color="4" fill="1" visible="no" active="no"/>
@@
 <part name="VR-5-4" library="parts" deviceset="L7805ACD2T-TR" device="" value="L7805"/>
 <part name="C_5V" library="parts" deviceset="CAPACITOR_POL" device="" value="0.33uF"/>
-<part name="5V_1" library="parts" deviceset="2-HOLES" device="SC3.81MM"/>
-<part name="5V_2" library="parts" deviceset="2-HOLES" device="SC3.81MM"/>
-<part name="5V_3" library="parts" deviceset="2-HOLES" device="SC3.81MM"/>
-<part name="5V_4" library="parts" deviceset="2-HOLES" device="SC3.81MM"/>
+<part name="5V_1" library="parts" deviceset="2-HOLES" device="SC3.81MM" value="SC3.81MM"/>
+<part name="5V_2" library="parts" deviceset="2-HOLES" device="SC3.81MM" value="SC3.81MM"/>
+<part name="5V_3" library="parts" deviceset="2-HOLES" device="SC3.81MM" value="SC3.81MM"/>
+<part name="5V_4" library="parts" deviceset="2-HOLES" device="SC3.81MM" value="SC3.81MM"/>
 <part name="C7" library="parts" deviceset="CAPACITOR_POL" device="" value="0.1uF"/>
 <part name="C8" library="parts" deviceset="CAPACITOR_POL" device="" value="0.1uF"/>
@@
 <part name="C10" library="parts" deviceset="CAPACITOR_POL" device="" value="0.1uF"/>
 <part name="C_ACT" library="parts" deviceset="CAPACITOR_POL" device="" value="0.33uF"/>
-<part name="12V_AM1" library="parts" deviceset="2-HOLES" device="SC3.81MM"/>
-<part name="12V_AM2" library="parts" deviceset="2-HOLES" device="SC3.81MM"/>
+<part name="12V_AM1" library="parts" deviceset="2-HOLES" device="SC3.81MM" value="SC3.81MM"/>
+<part name="12V_AM2" library="parts" deviceset="2-HOLES" device="SC3.81MM" value="SC3.81MM"/>
 <part name="C13" library="parts" deviceset="CAPACITOR_POL" device="" value="0.1uF"/>
 <part name="C14" library="parts" deviceset="CAPACITOR_POL" device="" value="0.1uF"/>
@@
 <part name="R5" library="parts" deviceset="RESISTOR" device="0207/2V" value="270R"/>
 <part name="R6" library="parts" deviceset="RESISTOR" device="0207/2V" value="1K"/>
-<part name="12V_SERVO1" library="parts" deviceset="2-HOLES" device="SC3.81MM"/>
+<part name="12V_SERVO1" library="parts" deviceset="2-HOLES" device="SC3.81MM" value="SC3.81MM"/>
 <part name="VR-S2" library="parts" deviceset="LM338T" device="-SINK" value="LM338T-SINK"/>
 <part name="C17" library="parts" deviceset="CAPACITOR_POL" device="" value="0.1uF"/>
 <part name="R7" library="parts" deviceset="RESISTOR" device="0207/2V" value="270R"/>
 <part name="R8" library="parts" deviceset="RESISTOR" device="0207/2V" value="1K"/>
-<part name="12V_SERVO2" library="parts" deviceset="2-HOLES" device="SC3.81MM"/>
+<part name="12V_SERVO2" library="parts" deviceset="2-HOLES" device="SC3.81MM" value="SC3.81MM"/>
 <part name="VR-S3" library="parts" deviceset="LM338T" device="-SINK" value="LM338T-SINK"/>
 <part name="C19" library="parts" deviceset="CAPACITOR_POL" device="" value="0.1uF"/>
 <part name="R9" library="parts" deviceset="RESISTOR" device="0207/2V" value="270R"/>
 <part name="R10" library="parts" deviceset="RESISTOR" device="0207/2V" value="1K"/>
-<part name="12V_SERVO3" library="parts" deviceset="2-HOLES" device="SC3.81MM"/>
+<part name="12V_SERVO3" library="parts" deviceset="2-HOLES" device="SC3.81MM" value="SC3.81MM"/>
 <part name="VR-S4" library="parts" deviceset="LM338T" device="-SINK" value="LM338T-SINK"/>
 <part name="C21" library="parts" deviceset="CAPACITOR_POL" device="" value="0.1uF"/>
 <part name="R11" library="parts" deviceset="RESISTOR" device="0207/2V" value="270R"/>
 <part name="R12" library="parts" deviceset="RESISTOR" device="0207/2V" value="1K"/>
-<part name="12V_SERVO4" library="parts" deviceset="2-HOLES" device="SC3.81MM"/>
+<part name="12V_SERVO4" library="parts" deviceset="2-HOLES" device="SC3.81MM" value="SC3.81MM"/>
 <part name="VR-S5" library="parts" deviceset="LM338T" device="-SINK" value="LM338T-SINK"/>
 <part name="C23" library="parts" deviceset="CAPACITOR_POL" device="" value="0.1uF"/>
 <part name="R13" library="parts" deviceset="RESISTOR" device="0207/2V" value="270R"/>
 <part name="R14" library="parts" deviceset="RESISTOR" device="0207/2V" value="1K"/>
-<part name="12V_SERVO5" library="parts" deviceset="2-HOLES" device="SC3.81MM"/>
+<part name="12V_SERVO5" library="parts" deviceset="2-HOLES" device="SC3.81MM" value="SC3.81MM"/>
 <part name="VR-S6" library="parts" deviceset="LM338T" device="-SINK" value="LM338T-SINK"/>
 <part name="C25" library="parts" deviceset="CAPACITOR_POL" device="" value="0.1uF"/>
 <part name="R15" library="parts" deviceset="RESISTOR" device="0207/2V" value="270R"/>
 <part name="R16" library="parts" deviceset="RESISTOR" device="0207/2V" value="1K"/>
-<part name="12V_SERVO6" library="parts" deviceset="2-HOLES" device="SC3.81MM"/>
+<part name="12V_SERVO6" library="parts" deviceset="2-HOLES" device="SC3.81MM" value="SC3.81MM"/>
 <part name="VR-12-2" library="parts" deviceset="L7812CD2T-TR" device="TO-263" value="L7812"/>
-<part name="VR-12-1" library="parts" deviceset="L7812CD2T-TR" device="TO-263" value="l7812"/>
+<part name="VR-12-1" library="parts" deviceset="L7812CD2T-TR" device="TO-263" value="L7812"/>
 <part name="C28" library="parts" deviceset="CAPACITOR_POL" device="" value="0.1uF"/>
 <part name="C_12V" library="parts" deviceset="CAPACITOR_POL" device="" value="0.33uF"/>
 <part name="C30" library="parts" deviceset="CAPACITOR_POL" device="" value="0.1uF"/>
-<part name="12V_REG-1" library="parts" deviceset="2-HOLES" device="SC3.81MM"/>
-<part name="12V_REG-2" library="parts" deviceset="2-HOLES" device="SC3.81MM"/>
+<part name="12V_REG-1" library="parts" deviceset="2-HOLES" device="SC3.81MM" value="SC3.81MM"/>
+<part name="12V_REG-2" library="parts" deviceset="2-HOLES" device="SC3.81MM" value="SC3.81MM"/>
 <part name="VR-A-1" library="parts" deviceset="LM1085IT" device="-SINK" value="LM1085-12V"/>
 <part name="VR-A-2" library="parts" deviceset="LM1085IT" device="-SINK" value="LM1085-12V"/>
-<part name="12V-1" library="parts" deviceset="2-HOLES" device="SC3.81MM"/>
-<part name="12V-2" library="parts" deviceset="2-HOLES" device="SC3.81MM"/>
-<part name="12V-3" library="parts" deviceset="2-HOLES" device="SC3.81MM"/>
-<part name="INPUT" library="parts" deviceset="3-HOLES" device=""/>
-<part name="OUTPUT" library="parts" deviceset="3-HOLES" device=""/>
+<part name="12V-1" library="parts" deviceset="2-HOLES" device="SC3.81MM" value="SC3.81MM"/>
+<part name="12V-2" library="parts" deviceset="2-HOLES" device="SC3.81MM" value="SC3.81MM"/>
+<part name="12V-3" library="parts" deviceset="2-HOLES" device="SC3.81MM" value="SC3.81MM"/>
+<part name="INPUT" library="parts" deviceset="3-HOLES" device="" value="SC3.8MM"/>
+<part name="OUTPUT" library="parts" deviceset="3-HOLES" device="" value="SC3.8MM"/>
 <part name="C_SERVO2" library="parts" deviceset="CAPACITOR_POL" device="" value="0.33uF"/>
 </parts>
