File: circuits/projects/Power_board/distribution_board.brd (EAGLE design)
At the start: 160 x 100 mm, 73 parts

Commit message: gittin the night away
Parts:
- 12V-1, 12V-2, 12V-3, 12V_AM1, 12V_AM2, 12V_REG-1, 12V_REG-2, 12V_SERVO1, 12V_SERVO2, 12V_SERVO3, 12V_SERVO4, 12V_SERVO5, 12V_SERVO6, 5V_1, 5V_2, 5V_3, 5V_4: value 2-HOLESSC3.81MM -> SC3.81MM
- INPUT, OUTPUT: value (none) -> SC3.8MM
- VR-12-1: value l7812 -> L7812
- moved U$3 2.54 mm to (138.4, 45.1)
Other:
- board text added: "Design & Production S. Martin"

Commit message: first board finished
Parts:
- removed U$1: (no value), parts:LOGO-ASSBOT
- moved C_SERVO2 12.8 mm to (36.8, 45.7)
- moved C14 8.03 mm to (19.1, 82.5)
- moved VR-A-2 6.84 mm to (15.2, 71.1)
- moved C_12V 5.43 mm to (62.9, 61.6)
- moved C_ACT 4.49 mm to (31.1, 60.3)
- moved U$4 2.62 mm to (10.2, 25.4)
- moved U$5 2.54 mm to (81.3, 41.3)
- moved VR-A-1 2.54 mm to (39.4, 71.1)
- moved C13 2.54 mm to (34.3, 82.5), turned to 0 degrees
- moved U$2 2.01 mm to (10.2, 26.0)
- moved U$3 1.80 mm to (139.7, 43.8)
- moved C_5V 1.27 mm to (124.5, 52.1)
Routing:
- net GND: track 766.4 -> 915.4 mm
- net 24V: track 364.0 -> 381.7 mm, vias 2 -> 4
- net 12V: track 342.6 -> 329.6 mm, vias 2 -> 3
- net N$3: track 55.0 -> 42.5 mm
- net N$25: track 39.1 -> 26.8 mm, vias 1 -> 0
- net N$37: track 39.1 -> 26.8 mm, vias 1 -> 0
- net N$34: track 39.1 -> 26.8 mm, vias 1 -> 0
- net N$31: track 39.0 -> 26.8 mm, vias 1 -> 0
- net N$28: track 39.0 -> 26.8 mm, vias 1 -> 0
- net N$23: track 35.7 -> 26.8 mm
- net N$13: track 26.8 -> 32.6 mm
- net N$15: track 39.0 -> 34.3 mm, vias 2 -> 1
- net N$18: track 37.7 -> 34.8 mm, vias 1 -> 0
- net N$14: track 29.2 -> 32.1 mm, vias 2 -> 1
- net N$17: track 31.7 -> 29.4 mm
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
Commit message: new shit
Routing:
- added copper zone on layer 1, net 12V
- added copper zone on layer 16, net 12V
- added copper zone on layer 1, net 24V
- added copper zone on layer 16, net 24V
- added copper zone on layer 16, net GND
- added copper zone on layer 16, net N$17
- added copper zone on layer 16, net N$18
- added copper zone on layer 16, net N$23
- added copper zone on layer 16, net N$25
- added copper zone on layer 16, net N$28
- added copper zone on layer 16, net N$31
- added copper zone on layer 16, net N$34
- added copper zone on layer 16, net N$37
