File: circuits/projects/Power_board/switch-fuses.sch (EAGLE design)
At the start: 18 parts

Commit message: more datasheets
Parts:
- B1, B2, FUSE-1, FUSE-2, V+, V-: value 2-HOLES2-HOLES-5.08MM -> 2-HOLES2.5MM; device parts:2-HOLES2-HOLES-5.08MM -> parts:2-HOLES2.5MM
- FUSE-LED1+, FUSE-LED1-, FUSE-LED2+, FUSE-LED2-, ON-LED1+, ON-LED1-, ON-LED2+, ON-LED2-: value 1-HOLE" -> 1-HOLE0.8MM; device parts:1-HOLE" -> parts:1-HOLE0.8MM
Changed lines of the file:
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@@
 <setting verticaltext="up"/>
 </settings>
-<grid distance="0.1" unitdist="inch" unit="inch" style="lines" multiple="1" display="yes" altdistance="0.01" altunitdist="inch" altunit="inch"/>
+<grid distance="0.1" unitdist="inch" unit="inch" style="lines" multiple="1" display="no" altdistance="0.01" altunitdist="inch" altunit="inch"/>
 <layers>
-<layer number="1" name="Top" color="4" fill="1" visible="no" active="no"/>
-<layer number="16" name="Bottom" color="1" fill="1" visible="no" active="no"/>
-<layer number="17" name="Pads" color="2" fill="1" visible="no" active="no"/>
-<layer number="18" name="Vias" color="2" fill="1" visible="no" active="no"/>
-<layer number="19" name="Unrouted" color="6" fill="1" visible="no" active="no"/>
-<layer number="20" name="Dimension" color="15" fill="1" visible="no" active="no"/>
-<layer number="21" name="tPlace" color="7" fill="1" visible="no" active="no"/>
-<layer number="22" name="bPlace" color="7" fill="1" visible="no" active="no"/>
-<layer number="23" name="tOrigins" color="15" fill="1" visible="no" active="no"/>
-<layer number="24" name="bOrigins" color="15" fill="1" visible="no" active="no"/>
-<layer number="25" name="tNames" color="7" fill="1" visible="no" active="no"/>
-<layer number="26" name="bNames" color="7" fill="1" visible="no" active="no"/>
-<layer number="27" name="tValues" color="7" fill="1" visible="no" active="no"/>
-<layer number="28" name="bValues" color="7" fill="1" visible="no" active="no"/>
+<layer number="1" name="Top" color="4" fill="1" visible="yes" active="no"/>
+<layer number="16" name="Bottom" color="1" fill="1" visible="yes" active="no"/>
+<layer number="17" name="Pads" color="2" fill="1" visible="yes" active="no"/>
+<layer number="18" name="Vias" color="2" fill="1" visible="yes" active="no"/>
+<layer number="19" name="Unrouted" color="6" fill="1" visible="yes" active="no"/>
+<layer number="20" name="Dimension" color="15" fill="1" visible="yes" active="no"/>
+<layer number="21" name="tPlace" color="7" fill="1" visible="yes" active="no"/>
+<layer number="22" name="bPlace" color="7" fill="1" visible="yes" active="no"/>
+<layer number="23" name="tOrigins" color="15" fill="1" visible="yes" active="no"/>
+<layer number="24" name="bOrigins" color="15" fill="1" visible="yes" active="no"/>
+<layer number="25" name="tNames" color="7" fill="1" visible="yes" active="no"/>
+<layer number="26" name="bNames" color="7" fill="1" visible="yes" active="no"/>
+<layer number="27" name="tValues" color="7" fill="1" visible="yes" active="no"/>
+<layer number="28" name="bValues" color="7" fill="1" visible="yes" active="no"/>
 <layer number="29" name="tStop" color="7" fill="3" visible="no" active="no"/>
 <layer number="30" name="bStop" color="7" fill="6" visible="no" active="no"/>
@@
 <layer number="35" name="tGlue" color="7" fill="4" visible="no" active="no"/>
 <layer number="36" name="bGlue" color="7" fill="5" visible="no" active="no"/>
-<layer number="37" name="tTest" color="7" fill="1" visible="no" active="no"/>
-<layer number="38" name="bTest" color="7" fill="1" visible="no" active="no"/>
+<layer number="37" name="tTest" color="7" fill="1" visible="yes" active="no"/>
+<layer number="38" name="bTest" color="7" fill="1" visible="yes" active="no"/>
 <layer number="39" name="tKeepout" color="4" fill="11" visible="no" active="no"/>
 <layer number="40" name="bKeepout" color="1" fill="11" visible="no" active="no"/>
@@
 <layer number="44" name="Drills" color="7" fill="1" visible="no" active="no"/>
 <layer number="45" name="Holes" color="7" fill="1" visible="no" active="no"/>
-<layer number="46" name="Milling" color="3" fill="1" visible="no" active="no"/>
-<layer number="47" name="Measures" color="7" fill="1" visible="no" active="no"/>
-<layer number="48" name="Document" color="7" fill="1" visible="no" active="no"/>
-<layer number="49" name="Reference" color="7" fill="1" visible="no" active="no"/>
-<layer number="50" name="dxf" color="7" fill="1" visible="no" active="no"/>
-<layer number="51" name="tDocu" color="7" fill="1" visible="no" active="no"/>
-<layer number="52" name="bDocu" color="7" fill="1" visible="no" active="no"/>
-<layer number="53" name="tGND_GNDA" color="7" fill="9" visible="no" active="no"/>
-<layer number="54" name="bGND_GNDA" color="1" fill="9" visible="no" active="no"/>
-<layer number="56" name="wert" color="7" fill="1" visible="no" active="no"/>
+<layer number="46" name="Milling" color="3" fill="1" visible="yes" active="no"/>
+<layer number="47" name="Measures" color="7" fill="1" visible="yes" active="no"/>
+<layer number="48" name="Document" color="7" fill="1" visible="yes" active="no"/>
+<layer number="49" name="Reference" color="7" fill="1" visible="yes" active="no"/>
+<layer number="50" name="dxf" color="7" fill="1" visible="yes" active="no"/>
+<layer number="51" name="tDocu" color="7" fill="1" visible="yes" active="no"/>
+<layer number="52" name="bDocu" color="7" fill="1" visible="yes" active="no"/>
+<layer number="53" name="tGND_GNDA" color="7" fill="9" visible="yes" active="no"/>
+<layer number="54" name="bGND_GNDA" color="1" fill="9" visible="yes" active="no"/>
+<layer number="56" name="wert" color="7" fill="1" visible="yes" active="no"/>
 <layer number="91" name="Nets" color="2" fill="1" visible="yes" active="yes"/>
 <layer number="92" name="Busses" color="1" fill="1" visible="yes" active="yes"/>
@@
 </classes>
 <parts>
-<part name="V+" library="parts" deviceset="2-HOLES" device="2-HOLES-5.08MM"/>
-<part name="V-" library="parts" deviceset="2-HOLES" device="2-HOLES-5.08MM"/>
-<part name="FUSE-2" library="parts" deviceset="2-HOLES" device="2-HOLES-5.08MM"/>
-<part name="FUSE-1" library="parts" deviceset="2-HOLES" device="2-HOLES-5.08MM"/>
+<part name="V+" library="parts" deviceset="2-HOLES" device="2.5MM" value="2-HOLES2.5MM"/>
+<part name="V-" library="parts" deviceset="2-HOLES" device="2.5MM" value="2-HOLES2.5MM"/>
+<part name="FUSE-2" library="parts" deviceset="2-HOLES" device="2.5MM" value="2-HOLES2.5MM"/>
+<part name="FUSE-1" library="parts" deviceset="2-HOLES" device="2.5MM" value="2-HOLES2.5MM"/>
 <part name="R1-FUSE" library="parts" deviceset="RESISTOR" device="0309/15" value="560R"/>
 <part name="R2-FUSE" library="parts" deviceset="RESISTOR" device="0309/15" value="560R"/>
-<part name="FUSE-LED1+" library="parts" deviceset="1-HOLE" device="&quot;"/>
-<part name="FUSE-LED2+" library="parts" deviceset="1-HOLE" device="&quot;"/>
-<part name="FUSE-LED1-" library="parts" deviceset="1-HOLE" device="&quot;"/>
-<part name="FUSE-LED2-" library="parts" deviceset="1-HOLE" device="&quot;"/>
-<part name="B1" library="parts" deviceset="2-HOLES" device="2-HOLES-5.08MM"/>
-<part name="B2" library="parts" deviceset="2-HOLES" device="2-HOLES-5.08MM"/>
+<part name="FUSE-LED1+" library="parts" deviceset="1-HOLE" device="0.8MM" value="1-HOLE0.8MM"/>
+<part name="FUSE-LED2+" library="parts" deviceset="1-HOLE" device="0.8MM" value="1-HOLE0.8MM"/>
+<part name="FUSE-LED1-" library="parts" deviceset="1-HOLE" device="0.8MM" value="1-HOLE0.8MM"/>
+<part name="FUSE-LED2-" library="parts" deviceset="1-HOLE" device="0.8MM" value="1-HOLE0.8MM"/>
+<part name="B1" library="parts" deviceset="2-HOLES" device="2.5MM" value="2-HOLES2.5MM"/>
+<part name="B2" library="parts" deviceset="2-HOLES" device="2.5MM" value="2-HOLES2.5MM"/>
 <part name="R1-ON" library="parts" deviceset="RESISTOR" device="0309/15" value="560R"/>
 <part name="R2-ON" library="parts" deviceset="RESISTOR" device="0309/15" value="560R"/>
-<part name="ON-LED1+" library="parts" deviceset="1-HOLE" device="&quot;"/>
-<part name="ON-LED2+" library="parts" deviceset="1-HOLE" device="&quot;"/>
-<part name="ON-LED1-" library="parts" deviceset="1-HOLE" device="&quot;"/>
-<part name="ON-LED2-" library="parts" deviceset="1-HOLE" device="&quot;"/>
+<part name="ON-LED1+" library="parts" deviceset="1-HOLE" device="0.8MM" value="1-HOLE0.8MM"/>
+<part name="ON-LED2+" library="parts" deviceset="1-HOLE" device="0.8MM" value="1-HOLE0.8MM"/>
+<part name="ON-LED1-" library="parts" deviceset="1-HOLE" device="0.8MM" value="1-HOLE0.8MM"/>
+<part name="ON-LED2-" library="parts" deviceset="1-HOLE" device="0.8MM" value="1-HOLE0.8MM"/>
 </parts>
 <sheets>

Commit message: new shit
Parts:
- removed B1, B2, FUSE-1, FUSE-2, V+, V-: 2-HOLES2.5MM, parts:2-HOLES2.5MM
- added B1_V+, B1_V+OUT, B1_V-, B1_V_OUT, B2_V+, B2_V+OUT, B2_V-, B2_V-OUT, F1_A, F1_B, F2_A, F2_B: 1-HOLE2.5MM, parts:1-HOLE2.5MM
Connections:
- net V+1: now also B2_V+OUT.1, F2_B.1; no longer B1.1, FUSE-1.2
- net V+2: now also B1_V+OUT.1, F1_B.1; no longer B2.2, FUSE-2.2
- net V-1: now also B1_V-.1, B1_V_OUT.1; no longer B1.2, V-.1
- net V-2: now also B2_V-.1, B2_V-OUT.1; no longer B2.1, V-.2
- net VIN1: now also B1_V+.1, F1_A.1; no longer FUSE-2.1, V+.2
- net VIN2: now also B2_V+.1, F2_A.1; no longer FUSE-1.1, V+.1
