File: circuits/projects/Power_board/battery_board.brd (EAGLE design)
At the start: 150 x 100 mm, 37 parts

Commit message: woowoooo
Parts:
- removed VR-MB1, VR-MB2, VR-MB3: LT323A, parts:TO220V-HEATSINK2
- added U$11, U$12, U$13: LD1085_3A-VREG, parts:TO220V
- moved C1_V1 9.52 mm to (57.1, 17.5)
- moved C2_V1 9.52 mm to (47.6, 17.5)
- moved C1_V2 9.21 mm to (93.7, 17.5)
- moved C1_V3 9.21 mm to (130.8, 17.5)
- moved C2_V2 9.21 mm to (84.5, 17.5)
- moved C2_V3 9.21 mm to (121.6, 17.5)
Connections:
- net 12V: now also U$11.3, U$12.3, U$13.3; no longer VR-MB1.1, VR-MB2.1, VR-MB3.1
- net GND: now also U$11.1, U$12.1, U$13.1; no longer VR-MB1.2, VR-MB2.2, VR-MB3.2
- net N$15: now also U$12.2; no longer VR-MB2.3
- net N$17: now also U$11.2; no longer VR-MB1.3
- net N$8: now also U$13.2; no longer VR-MB3.3
Routing:
- net 12V: track 284.9 -> 239.2 mm
- net GND: track 511.3 -> 531.1 mm
- net N$8: track 25.0 -> 23.5 mm
- net N$17: track 24.9 -> 23.8 mm
- net N$15: track 24.9 -> 23.9 mm
