File: circuits/projects/Power_board/battery_board.brd (EAGLE design)
At the start: 150 x 100 mm, 37 parts

Commit message: board
Parts:
- moved U$8 7.43 mm to (108.0, 50.5)
Routing:
- net 12V: track 239.2 -> 251.0 mm

Commit message: wooo
Parts:
- U$11, U$12, U$13: device parts:TO220V -> parts:TO220V-HEATSINK2
- moved U$8 2.01 mm to (106.0, 51.1)
Routing:
- net 12V: track 251.0 -> 249.9 mm
Changed lines of the file:
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@@
 <grid distance="25" unitdist="mil" unit="mil" style="lines" multiple="1" display="yes" altdistance="6.25" altunitdist="mil" altunit="mil"/>
 <layers>
-<layer number="1" name="Top" color="4" fill="1" visible="no" active="yes"/>
+<layer number="1" name="Top" color="4" fill="1" visible="yes" active="yes"/>
 <layer number="2" name="Route2" color="1" fill="3" visible="no" active="no"/>
 <layer number="3" name="Route3" color="4" fill="3" visible="no" active="no"/>
@@
 <layer number="19" name="Unrouted" color="6" fill="1" visible="yes" active="yes"/>
 <layer number="20" name="Dimension" color="15" fill="1" visible="yes" active="yes"/>
-<layer number="21" name="tPlace" color="7" fill="1" visible="yes" active="yes"/>
-<layer number="22" name="bPlace" color="7" fill="1" visible="yes" active="yes"/>
-<layer number="23" name="tOrigins" color="15" fill="1" visible="yes" active="yes"/>
+<layer number="21" name="tPlace" color="7" fill="1" visible="no" active="yes"/>
+<layer number="22" name="bPlace" color="7" fill="1" visible="no" active="yes"/>
+<layer number="23" name="tOrigins" color="15" fill="1" visible="no" active="yes"/>
 <layer number="24" name="bOrigins" color="15" fill="1" visible="yes" active="yes"/>
-<layer number="25" name="tNames" color="7" fill="1" visible="yes" active="yes"/>
-<layer number="26" name="bNames" color="7" fill="1" visible="yes" active="yes"/>
-<layer number="27" name="tValues" color="7" fill="1" visible="yes" active="yes"/>
-<layer number="28" name="bValues" color="7" fill="1" visible="yes" active="yes"/>
+<layer number="25" name="tNames" color="7" fill="1" visible="no" active="yes"/>
+<layer number="26" name="bNames" color="7" fill="1" visible="no" active="yes"/>
+<layer number="27" name="tValues" color="7" fill="1" visible="no" active="yes"/>
+<layer number="28" name="bValues" color="7" fill="1" visible="no" active="yes"/>
 <layer number="29" name="tStop" color="7" fill="3" visible="yes" active="yes"/>
-<layer number="30" name="bStop" color="7" fill="6" visible="no" active="yes"/>
+<layer number="30" name="bStop" color="7" fill="6" visible="yes" active="yes"/>
 <layer number="31" name="tCream" color="7" fill="4" visible="no" active="yes"/>
 <layer number="32" name="bCream" color="7" fill="5" visible="no" active="yes"/>
@@
 <layer number="39" name="tKeepout" color="4" fill="11" visible="no" active="yes"/>
 <layer number="40" name="bKeepout" color="1" fill="11" visible="no" active="yes"/>
-<layer number="41" name="tRestrict" color="4" fill="10" visible="yes" active="yes"/>
-<layer number="42" name="bRestrict" color="1" fill="10" visible="yes" active="yes"/>
+<layer number="41" name="tRestrict" color="4" fill="10" visible="no" active="yes"/>
+<layer number="42" name="bRestrict" color="1" fill="10" visible="no" active="yes"/>
 <layer number="43" name="vRestrict" color="2" fill="10" visible="no" active="yes"/>
 <layer number="44" name="Drills" color="7" fill="1" visible="no" active="yes"/>
@@
 <layer number="111" name="LPC17xx" color="7" fill="1" visible="no" active="yes"/>
 <layer number="112" name="tSilk" color="7" fill="1" visible="no" active="yes"/>
-<layer number="113" name="IDFDebug" color="7" fill="1" visible="yes" active="yes"/>
+<layer number="113" name="IDFDebug" color="7" fill="1" visible="no" active="yes"/>
 <layer number="116" name="Patch_BOT" color="9" fill="4" visible="no" active="yes"/>
 <layer number="121" name="_tplace" color="14" fill="1" visible="yes" active="yes"/>
-<layer number="122" name="_bplace" color="14" fill="1" visible="yes" active="yes"/>
+<layer number="122" name="_bplace" color="14" fill="1" visible="no" active="yes"/>
 <layer number="123" name="tTestmark" color="7" fill="1" visible="no" active="yes"/>
 <layer number="124" name="bTestmark" color="7" fill="1" visible="no" active="yes"/>
@@
 <layer number="145" name="DrillLegend_01-16" color="2" fill="9" visible="no" active="yes"/>
 <layer number="146" name="DrillLegend_01-20" color="3" fill="9" visible="no" active="yes"/>
-<layer number="150" name="Notes" color="7" fill="1" visible="yes" active="yes"/>
+<layer number="150" name="Notes" color="7" fill="1" visible="no" active="yes"/>
 <layer number="151" name="HeatSink" color="7" fill="1" visible="no" active="yes"/>
 <layer number="152" name="_bDocu" color="7" fill="1" visible="no" active="yes"/>
-<layer number="153" name="FabDoc1" color="7" fill="1" visible="yes" active="yes"/>
-<layer number="154" name="FabDoc2" color="7" fill="1" visible="yes" active="yes"/>
-<layer number="155" name="FabDoc3" color="7" fill="1" visible="yes" active="yes"/>
+<layer number="153" name="FabDoc1" color="7" fill="1" visible="no" active="yes"/>
+<layer number="154" name="FabDoc2" color="7" fill="1" visible="no" active="yes"/>
+<layer number="155" name="FabDoc3" color="7" fill="1" visible="no" active="yes"/>
 <layer number="199" name="Contour" color="7" fill="1" visible="no" active="yes"/>
 <layer number="200" name="200bmp" color="1" fill="10" visible="no" active="yes"/>
@@
 <text x="90.805" y="93.6625" size="2.54" layer="121" font="vector" ratio="14" rot="R90" align="bottom-center">B1</text>
 <text x="58.1025" y="93.345" size="2.54" layer="121" font="vector" ratio="14" rot="R90" align="bottom-center">B2</text>
-<text x="4.445" y="38.4175" size="2.54" layer="16" font="vector" ratio="13" rot="MR180">Design &amp; Production
+<text x="4.445" y="42.2275" size="2.54" layer="16" font="vector" ratio="13" rot="MR180">Design &amp; Production
 S. Martin</text>
 <text x="10.16" y="60.325" size="1.778" layer="121" font="vector" ratio="14" rot="R180" align="bottom-center">MOTOR 2</text>
@@
 <element name="U$6" library="parts" package="3,0" value="" x="5" y="5"/>
 <element name="U$7" library="parts" package="LOGO-ASSBOT" value="" x="42.2275" y="16.8275" rot="SMR0"/>
-<element name="U$8" library="parts" package="LOGO-SYNCHROTRON" value="" x="107.95" y="50.4825" rot="MR0"/>
+<element name="U$8" library="parts" package="LOGO-SYNCHROTRON" value="" x="106.045" y="51.1175" rot="MR0"/>
 <element name="U$2" library="parts" package="LOGO-ASSBOT-SILK" value="" x="40.64" y="40.005" rot="SR0"/>
 <element name="FUSE-M2" library="parts" package="SCREWTERMINAL-5MM-2" value="3A" x="40.64" y="93.0275" rot="R180"/>
@@
 <element name="U$1" library="parts" package="LOGO-SYNCHROTRON" value="" x="128.905" y="43.4975"/>
 <element name="U$9" library="parts" package="LOGO-ASSBOT" value="" x="4.7625" y="12.3825" rot="SR0"/>
-<element name="U$11" library="parts" package="TO220V" value="LD1085_3A-VREG" x="52.705" y="30.1625"/>
-<element name="U$12" library="parts" package="TO220V" value="LD1085_3A-VREG" x="89.535" y="30.1625"/>
-<element name="U$13" library="parts" package="TO220V" value="LD1085_3A-VREG" x="126.365" y="30.1625"/>
+<element name="U$11" library="parts" package="TO220V-HEATSINK2" value="LD1085_3A-VREG" x="52.705" y="30.1625"/>
+<element name="U$12" library="parts" package="TO220V-HEATSINK2" value="LD1085_3A-VREG" x="89.535" y="30.1625"/>
+<element name="U$13" library="parts" package="TO220V-HEATSINK2" value="LD1085_3A-VREG" x="126.365" y="30.1625"/>
 </elements>
 <signals>
@@
 <wire x1="128.905" y1="31.115" x2="121.285" y2="40.005" width="1.778" layer="16"/>
 <wire x1="121.285" y1="40.005" x2="92.075" y2="40.005" width="1.778" layer="16"/>
-<wire x1="55.245" y1="27.6225" x2="56.515" y2="27.6225" width="1.778" layer="16"/>
-<wire x1="56.515" y1="27.6225" x2="56.515" y2="35.56" width="1.778" layer="16"/>
-<wire x1="56.515" y1="35.56" x2="61.9125" y2="40.005" width="1.778" layer="16"/>
+<wire x1="55.245" y1="27.94" x2="55.245" y2="34.925" width="1.778" layer="16"/>
+<wire x1="55.245" y1="34.925" x2="61.9125" y2="40.005" width="1.778" layer="16"/>
 <wire x1="61.9125" y1="40.005" x2="92.075" y2="40.005" width="1.778" layer="16"/>
 <wire x1="54.61" y1="17.4625" x2="54.61" y2="18.415" width="1.27" layer="16"/>
-<wire x1="54.61" y1="18.415" x2="55.88" y2="19.685" width="1.27" layer="16"/>
-<wire x1="55.88" y1="19.685" x2="55.88" y2="26.9875" width="1.27" layer="16"/>
-<wire x1="55.88" y1="26.9875" x2="55.245" y2="27.6225" width="1.778" layer="16"/>
+<wire x1="54.61" y1="18.415" x2="55.245" y2="19.05" width="1.27" layer="16"/>
+<wire x1="55.245" y1="19.05" x2="55.245" y2="27.6225" width="1.27" layer="16"/>
 <wire x1="91.1225" y1="17.4625" x2="92.075" y2="18.415" width="1.27" layer="16"/>
 <wire x1="92.075" y1="18.415" x2="92.075" y2="27.6225" width="1.27" layer="16"/>
 <wire x1="128.27" y1="17.4625" x2="128.905" y2="18.0975" width="1.27" layer="16"/>
 <wire x1="128.905" y1="18.0975" x2="128.905" y2="27.6225" width="1.27" layer="16"/>
+<wire x1="55.245" y1="27.6225" x2="55.245" y2="27.94" width="1.27" layer="16"/>
 </signal>
 <signal name="MASK">

Commit message: zippity boo
Parts:
- removed D1-12V: 30A, parts:TO22-DIODE-H
- moved U$8 48.7 mm to (58.4, 61.3)
- moved U$9 45.3 mm to (40.6, 40.0)
- moved U$1 34.5 mm to (99.7, 61.9)
- moved U$7 33.4 mm to (68.3, 37.8)
Connections:
- removed net N$1: BATTERY1.2, BATTERY2.1, D1-12V.P$1, TEST.2
- removed net N$4: BATTERY2.2, D3-24V.P$1, TEST.3
- new net N$5: BATTERY1.2, BATTERY2.1, R3.1, TEST.2
- net 12V: now also BATTERY2.2, D3-24V.P$1, TEST.3; no longer D1-12V.P$2, OUTPUT-SHAFT.3, OUTPUT.3, R3.1
- net 24V: now also OUTPUT-SHAFT.3, OUTPUT.3
Routing:
- net N$5: track 0.00 -> 76.3 mm
- net N$1: track 58.0 -> 0.00 mm
- net 12V: track 249.9 -> 193.5 mm
- net GND: track 531.1 -> 483.6 mm, vias 4 -> 6
- net N$4: track 33.2 -> 0.00 mm
- net 24V: track 208.3 -> 237.2 mm, vias 3 -> 7
- net N$8: track 23.1 -> 34.3 mm
- net N$17: track 23.8 -> 34.3 mm
- net N$15: track 23.9 -> 34.1 mm
- net N$10: track 44.0 -> 42.8 mm, vias 2 -> 0
- net N$9: track 70.1 -> 70.7 mm, vias 2 -> 0
- added copper zone on layer 1, net GND
- removed copper zone on layer 1, net MASK
