File: circuits/projects/LINbus/injector.brd (EAGLE design)
At the start: 75 x 50 mm, 34 parts, among them J4 ICSP, U1 ATA6631, U2 ATMEGA328, U3 ATA6631, X1 16MHz

Commit message: Poorly Rooted V1
Parts:
- moved J3 55.7 mm to (4.06, 24.4), turned to 270 degrees
- moved R1 38.6 mm to (40.0, 29.5)
- moved D7 34.9 mm to (62.4, 6.60)
- moved R2 33.4 mm to (44.9, 29.4)
- moved D1 27.6 mm to (13.5, 47.1), turned to 180 degrees
- moved R6 24.8 mm to (43.8, 4.70)
- moved X1 21.3 mm to (32.1, 14.2)
- moved D5 20.3 mm to (62.4, 15.5)
- moved C1 19.3 mm to (10.0, 24.8)
- moved R5 18.5 mm to (47.9, 8.76)
- moved D2 18.3 mm to (13.5, 44.3), turned to 180 degrees
- moved D3 17.2 mm to (18.5, 36.4), turned to 270 degrees
- moved R8 14.0 mm to (20.3, 9.78)
- moved J4 13.0 mm to (62.1, 23.1), turned to 0 degrees
- moved U3 12.7 mm to (62.0, 33.5)
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Routing:
- net LIN2_TX: track 0.00 -> 55.4 mm, vias 0 -> 4
- net S-5V: track 72.1 -> 28.8 mm
- net LIN1_TX: track 0.00 -> 41.2 mm, vias 0 -> 2
- net DTR: track 47.9 -> 8.76 mm
- net +5V: track 109.5 -> 144.8 mm, vias 3 -> 2
- net MOSI/LIN_ERR: track 0.00 -> 34.2 mm, vias 0 -> 1
- net LIN1_RX: track 0.00 -> 33.8 mm, vias 0 -> 2
- net N$3: track 45.4 -> 18.8 mm
- net SECONDARY_5V: track 36.7 -> 63.1 mm, vias 2 -> 3
- net N$6: track 71.6 -> 45.7 mm, vias 1 -> 2
- net LIN2_RX: track 0.00 -> 24.8 mm
- net MISO/LIN_DATA: track 0.00 -> 22.8 mm, vias 0 -> 1
- net SCK: track 0.00 -> 18.3 mm, vias 0 -> 1
- net GND: track 242.7 -> 230.2 mm, vias 1 -> 6
- net RXI: track 46.7 -> 35.6 mm
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