File: circuits/projects/head_led/pig_led.brd (EAGLE design)
At the start: 50 x 30 mm, 12 parts

Commit message: pig skull led board complete
Parts:
- JP1: device iStivi - Header-Connector:SCREWTERMINAL-3.5MM-2 -> parts:SCREWTERMINAL-3.5MM-2
- R1, R2, R3, R4, R5, R6, R7, R8: device iStivi - RCLD:0207/10 -> parts:0207/10
- U$1: value M08X2 -> M08X2-0.3MMDRILL; device iStivi - Header-Connector:2X8 -> parts:2X8
Routing:
- net GND: track 38.3 -> 0.00 mm
- net VCC: track 32.1 -> 0.00 mm
