File: circuits/projects/head_led/pig_led.sch (EAGLE design)
At the start: 10 parts

Commit message: pig skull led board complete
Parts:
- JP1: device iStivi - Header-Connector:M023.5MM -> parts:M023.5MM
- R1, R2, R3, R4, R5, R6, R7, R8: device iStivi - RCLD:RESISTOR0207/10 -> parts:RESISTOR0207/10
- U$1: value M08X2 -> M08X2-0.3MMDRILL; device iStivi - Header-Connector:M08X2 -> parts:M08X2-0.3MMDRILL
