File: circuits/projects/battery_display/battery_monitor.sch (EAGLE design)
At the start: 20 parts, among them IC1 7805T, U1 ATMEGA328P_PDIP

Commit message: woowoooo
Parts:
- added C3: 100nF, iStivi - RCLD:CAPACITOR050-025X075
- added JP1: (no value), iStivi - Header-Connector:M06LONGPADS
Connections:
- new net N$7: C3.2, JP1.6
- net GND: now also JP1.1, JP1.2
- net N$6: now also C3.1
- net RX: now also JP1.4
- net TX: now also JP1.5
Changed lines of the file:
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@@
 <part name="GND5" library="parts" deviceset="GND" device=""/>
 <part name="LCD-POW" library="parts" deviceset="M03" device="PTH"/>
+<part name="JP1" library="iStivi - Header-Connector" deviceset="M06" device="LONGPADS"/>
+<part name="C3" library="iStivi - RCLD" deviceset="CAPACITOR" device="050-025X075" value="100nF"/>
 </parts>
 <sheets>
@@
 <instance part="GND5" gate="1" x="-35.56" y="35.56"/>
 <instance part="LCD-POW" gate="G$1" x="-15.24" y="5.08" rot="R90"/>
+<instance part="JP1" gate="G$1" x="157.48" y="91.44" rot="R180"/>
+<instance part="C3" gate="G$1" x="66.04" y="91.44" rot="R90"/>
 </instances>
 <busses>
@@
 <pinref part="GND4" gate="1" pin="GND"/>
 <pinref part="R1" gate="G$1" pin="1"/>
-<wire x1="116.84" y1="66.04" x2="116.84" y2="78.74" width="0.1524" layer="91"/>
+<wire x1="116.84" y1="66.04" x2="116.84" y2="76.2" width="0.1524" layer="91"/>
+<pinref part="JP1" gate="G$1" pin="1"/>
+<wire x1="116.84" y1="76.2" x2="116.84" y2="78.74" width="0.1524" layer="91"/>
+<wire x1="152.4" y1="96.52" x2="134.62" y2="96.52" width="0.1524" layer="91"/>
+<wire x1="134.62" y1="96.52" x2="121.92" y2="96.52" width="0.1524" layer="91"/>
+<wire x1="121.92" y1="96.52" x2="121.92" y2="76.2" width="0.1524" layer="91"/>
+<wire x1="121.92" y1="76.2" x2="116.84" y2="76.2" width="0.1524" layer="91"/>
+<junction x="116.84" y="76.2"/>
+<pinref part="JP1" gate="G$1" pin="2"/>
+<wire x1="152.4" y1="93.98" x2="134.62" y2="93.98" width="0.1524" layer="91"/>
+<wire x1="134.62" y1="93.98" x2="134.62" y2="96.52" width="0.1524" layer="91"/>
+<junction x="134.62" y="96.52"/>
 </segment>
 <segment>
@@
 <pinref part="RX/TX" gate="G$1" pin="1"/>
 <wire x1="152.4" y1="60.96" x2="142.24" y2="60.96" width="0.1524" layer="91"/>
-<wire x1="142.24" y1="60.96" x2="132.08" y2="50.8" width="0.1524" layer="91"/>
+<wire x1="142.24" y1="60.96" x2="137.16" y2="55.88" width="0.1524" layer="91"/>
+<pinref part="JP1" gate="G$1" pin="4"/>
+<wire x1="137.16" y1="55.88" x2="132.08" y2="50.8" width="0.1524" layer="91"/>
+<wire x1="152.4" y1="88.9" x2="137.16" y2="88.9" width="0.1524" layer="91"/>
+<wire x1="137.16" y1="88.9" x2="137.16" y2="55.88" width="0.1524" layer="91"/>
+<junction x="137.16" y="55.88"/>
 </segment>
 </net>
@@
 <pinref part="RX/TX" gate="G$1" pin="2"/>
 <wire x1="152.4" y1="58.42" x2="142.24" y2="58.42" width="0.1524" layer="91"/>
-<wire x1="142.24" y1="58.42" x2="132.08" y2="48.26" width="0.1524" layer="91"/>
+<wire x1="142.24" y1="58.42" x2="139.7" y2="55.88" width="0.1524" layer="91"/>
+<pinref part="JP1" gate="G$1" pin="5"/>
+<wire x1="139.7" y1="55.88" x2="132.08" y2="48.26" width="0.1524" layer="91"/>
+<wire x1="152.4" y1="86.36" x2="139.7" y2="86.36" width="0.1524" layer="91"/>
+<wire x1="139.7" y1="86.36" x2="139.7" y2="55.88" width="0.1524" layer="91"/>
+<junction x="139.7" y="55.88"/>
 </segment>
 </net>
@@
 <wire x1="-35.56" y1="55.88" x2="-35.56" y2="60.96" width="0.1524" layer="91"/>
 <junction x="-35.56" y="60.96"/>
+<pinref part="C3" gate="G$1" pin="1"/>
+<wire x1="63.5" y1="91.44" x2="40.64" y2="91.44" width="0.1524" layer="91"/>
+<wire x1="40.64" y1="91.44" x2="40.64" y2="73.66" width="0.1524" layer="91"/>
+<junction x="40.64" y="73.66"/>
 </segment>
 </net>
@@
 </segment>
 </net>
+<net name="N$7" class="0">
+<segment>
+<pinref part="JP1" gate="G$1" pin="6"/>
+<wire x1="152.4" y1="83.82" x2="127" y2="83.82" width="0.1524" layer="91"/>
+<wire x1="127" y1="83.82" x2="127" y2="93.98" width="0.1524" layer="91"/>
+<wire x1="127" y1="93.98" x2="119.38" y2="93.98" width="0.1524" layer="91"/>
+<wire x1="119.38" y1="93.98" x2="119.38" y2="96.52" width="0.1524" layer="91"/>
+<pinref part="C3" gate="G$1" pin="2"/>
+<wire x1="119.38" y1="96.52" x2="71.12" y2="96.52" width="0.1524" layer="91"/>
+<wire x1="71.12" y1="96.52" x2="71.12" y2="91.44" width="0.1524" layer="91"/>
+</segment>
+</net>
