File: circuits/projects/battery_display/battery_monitor.brd (EAGLE design)
At the start: 100 x 77 mm, 26 parts, among them IC1 7805T, U1 ATMEGA328P_PDIP

Commit message: some boards updated
Routing:
- net RS: track 38.1 -> 45.9 mm
- net E: track 41.4 -> 45.8 mm
- net N$9: track 55.0 -> 57.6 mm
- net R/W: track 46.7 -> 48.7 mm
- net D7: track 64.1 -> 65.5 mm
- net RX: track 51.3 -> 52.5 mm
- net D5: track 34.5 -> 35.7 mm
- net TX: track 43.3 -> 44.3 mm
- net N$1: track 15.9 -> 16.5 mm

Commit message: woowoooo
Parts:
- added C3: 100nF, iStivi - RCLD:C050-025X075
- added JP1: (no value), iStivi - Header-Connector:1X06_LONGPADS
- moved LCD-POW 20.3 mm to (49.5, 11.4)
- moved LCD_2 15.2 mm to (61.0, 11.4)
- moved LCD_1 11.4 mm to (71.1, 11.4)
- moved U$8 5.24 mm to (19.1, 53.3)
- moved U$2 1.27 mm to (12.7, 20.3)
Connections:
- new net N$7: C3.2, JP1.6
- net GND: now also JP1.1, JP1.2
- net N$6: now also C3.1
- net RX: now also JP1.4
- net TX: now also JP1.5
Routing:
- net TX: track 44.3 -> 73.7 mm
- net D7: track 65.5 -> 42.6 mm, vias 0 -> 2
- net D5: track 35.7 -> 51.6 mm
- net RS: track 45.9 -> 30.5 mm, vias 2 -> 0
- net V0: track 186.9 -> 175.1 mm, vias 2 -> 3
- net N$7: track 0.00 -> 10.7 mm
- net R/W: track 48.7 -> 39.4 mm, vias 2 -> 0
- net D4: track 22.5 -> 30.5 mm, vias 0 -> 2
- net RX: track 52.5 -> 56.7 mm, vias 0 -> 2
- net GND: track 167.9 -> 171.9 mm
- net N$4: track 56.9 -> 54.2 mm
- net N$9: track 57.6 -> 55.0 mm
- net D6: track 42.3 -> 44.7 mm
- net N$6: track 33.8 -> 31.4 mm
- net E: track 45.8 -> 44.1 mm, vias 2 -> 0
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- removed copper zone on layer 1, net GND
- removed copper zone on layer 16, net GND

Commit message: board
Parts:
- moved R1 5.08 mm to (45.7, 54.6)
- moved R2 3.81 mm to (48.3, 49.5)
- moved U$1 1.27 mm to (48.3, 21.6)
Routing:
- net E: track 44.1 -> 79.8 mm
- net GND: track 171.9 -> 189.4 mm
- net V0: track 175.1 -> 191.8 mm
- net N$9: track 55.0 -> 68.1 mm
- net N$8: track 33.5 -> 45.0 mm
- net TX: track 73.7 -> 82.6 mm
- net D4: track 30.5 -> 36.9 mm
- net R/W: track 39.4 -> 44.3 mm
- net D7: track 42.6 -> 46.2 mm
- net N$6: track 31.4 -> 34.3 mm
- net D6: track 44.7 -> 47.4 mm
- net RS: track 30.5 -> 32.8 mm
- net N$2: track 8.89 -> 7.62 mm
- net D5: track 51.6 -> 52.6 mm
- net RX: track 56.7 -> 57.5 mm

Commit message: wooo
Routing:
- net R/W: track 44.3 -> 43.8 mm
Changed lines of the file:
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@@
 <setting verticaltext="up"/>
 </settings>
-<grid distance="0.05" unitdist="inch" unit="mil" style="lines" multiple="1" display="yes" altdistance="0.025" altunitdist="inch" altunit="mil"/>
+<grid distance="1" unitdist="mm" unit="mm" style="lines" multiple="1" display="yes" altdistance="0.025" altunitdist="inch" altunit="mil"/>
 <layers>
 <layer number="1" name="Top" color="4" fill="1" visible="yes" active="yes"/>
@@
 <wire x1="57.15" y1="40.64" x2="55.88" y2="39.37" width="1.27" layer="16"/>
 <wire x1="64.77" y1="40.64" x2="57.15" y2="40.64" width="1.27" layer="16"/>
-<wire x1="67.31" y1="39.37" x2="64.77" y2="40.64" width="1.27" layer="16"/>
-<wire x1="67.31" y1="17.78" x2="67.31" y2="39.37" width="1.27" layer="16"/>
+<wire x1="67.31" y1="38.1" x2="64.77" y2="40.64" width="1.27" layer="16"/>
+<wire x1="67.31" y1="17.78" x2="67.31" y2="38.1" width="1.27" layer="16"/>
 <wire x1="63.5" y1="11.43" x2="63.5" y2="13.97" width="1.27" layer="16"/>
 <wire x1="63.5" y1="13.97" x2="67.31" y2="17.78" width="1.27" layer="16"/>
